Commit message: Fix mass, inertia and max wheel velocity

File: car_description/urdf/body.xacro (robot description, xacro)
@@ -18,8 +18,8 @@
             </collision>
             <inertial>
-                <mass value="1"/>
-                <inertia ixx="0.001632" ixy="0.000000" ixz="0.0000000"
-                                        iyy="0.012465" iyz="0.0000000"
-                                                       izz="0.0132333"/>
+                <mass value="3.3"/>
+                <inertia ixx="0.005386" ixy="0.000000" ixz="0.00000"
+                                        iyy="0.041136" iyz="0.00000"
+                                                       izz="0.04367"/>
             </inertial>
         </link>

File: car_description/urdf/car.xacro (robot description, xacro)
@@ -17,5 +17,5 @@
             <i>0.0</i>
             <d>0.0</d>
-            <max_velocity>15.0</max_velocity>
+            <max_velocity>17.0</max_velocity>
         </plugin>
     </gazebo>

File: car_description/urdf/wheel.xacro (robot description, xacro)
@@ -20,8 +20,8 @@
             </collision>
             <inertial>
-                <mass value="0.1"/>
-                <inertia ixx="0.00012923" ixy="0.00000000" ixz="0000000"
-                                          iyy="0.00012923" iyz="0000000"
-                                                           izz="0.00315"/>
+                <mass value="0.150"/>
+                <inertia ixx="0.00019384" ixy="0.00000000" ixz="00000000"
+                                          iyy="0.00019384" iyz="00000000"
+                                                           izz="0.004725"/>
             </inertial>
         </link>

Commit message: Исправления и добавления  - добавил модель трека  - заменил меши машинки stl на collada и добавил им цвета  - добавил модельку камеры

File: car_description/urdf/body.xacro (robot description, xacro)
@@ -5,9 +5,6 @@
             <visual>
                 <geometry>
-                    <mesh filename="package://car_description/meshes/body.stl"/>
+                    <mesh filename="package://car_description/meshes/body.dae"/>
                 </geometry>
-                <material name="white">
-                    <color rgba="0.7 0.7 0.7 1.0"/>
-                </material>
             </visual>
             <collision>
@@ -24,7 +21,4 @@
             </inertial>
         </link>
-        <gazebo reference="base_link">
-            <material>Gazebo/Grey</material>
-        </gazebo>
     </xacro:macro>
 </robot>

File: car_description/urdf/camera.xacro (robot description, xacro)
@@ -2,8 +2,6 @@
 <robot xmlns:xacro="http://www.ros.org/wiki/xacro">
 	<xacro:macro name="my_camera">
-	  <!-- Camera -->
 	  <link name="camera_link">
 	    <collision>
-	      <!--<origin xyz="0.190 0 ${camera_size}" rpy="0 0 0"/>-->
 	      <geometry>
 	        <box size="0.007 0.03 0.03"/>
@@ -11,7 +9,6 @@
 	    </collision>
 	    <visual>
-	      <!--<origin xyz="0.190 0 ${camera_size}" rpy="0 0 0"/>-->
 	      <geometry>
-	        <box size="0.007 0.03 0.03"/>
+	        <mesh filename="package://car_description/meshes/camera.dae"/>
 	      </geometry>
 	      <material name="red"/>
@@ -19,5 +16,4 @@
 	    <inertial>
 	      <mass value="1e-5" />
-	      <!--<origin xyz="0.190 0 ${camera_size}" rpy="0 0 0"/>-->
 	      <inertia ixx="1e-6" ixy="0" ixz="0" iyy="1e-6" iyz="0" izz="1e-6" />
 	    </inertial>
@@ -25,6 +21,5 @@
 	  <joint name="camera_joint" type="fixed">
 	    <axis xyz="0 0 0" />
-	    <!--<origin xyz="0.1935 0 0.012" rpy="0 0 0"/>-->
-	    <origin xyz="-0.1920 0 0.012" rpy="3.14 3.14 0"/>
+	    <origin xyz="0.185 0 0.012" rpy="0 0 0"/>
 	    <parent link="base_link"/>
 	    <child link="camera_link"/>

File: car_description/urdf/car.xacro (robot description, xacro)
@@ -6,5 +6,5 @@
     <xacro:include filename="camera.xacro"/>
     <xacro:property name="wheel_stride" value="0.150" />
-    <xacro:property name="camera_size" value="0.03" /> <!-- Size of square 'camera' box -->
+    <xacro:property name="camera_size" value="0.03" />
     <xacro:body/>
     <xacro:wheel parent="base_link" side="left" x_pos="${-wheel_stride}" name="wheel_1_left"/>

File: car_description/urdf/left_right.xacro (robot description, xacro)
@@ -4,8 +4,8 @@
     <xacro:macro name="left_right" params="side">
         <xacro:if value="${side == 'left'}">
-            <xacro:property scope="parent" name="x_sign" value="-1" />
+            <xacro:property scope="parent" name="x_sign" value="1" />
         </xacro:if>
         <xacro:if value="${side == 'right'}">
-            <xacro:property scope="parent" name="x_sign" value="1" />
+            <xacro:property scope="parent" name="x_sign" value="-1" />
         </xacro:if>
     </xacro:macro>

File: car_description/urdf/wheel.xacro (robot description, xacro)
@@ -7,9 +7,6 @@
             <visual>
                 <geometry>
-                    <mesh filename="package://car_description/meshes/wheel_${side}.stl"/>
+                    <mesh filename="package://car_description/meshes/wheel_${side}.dae"/>
                 </geometry>
-                <material name="black">
-                    <color rgba="0.175 .175 .175 1.0"/>
-                </material>
             </visual>
             <collision>
@@ -26,9 +23,4 @@
             </inertial>
         </link>
-        <gazebo reference="${name}">
-            <material>Gazebo/DarkGrey</material>
-            <!--<mu1>0.6</mu1>
-            <mu2>0.6</mu2>-->
-        </gazebo>
         <joint name="${name}_joint" type="continuous">
             <parent link="${parent}"/>
