Commit message: Moved camera to car's front

File: car_description/urdf/camera.xacro (robot description, xacro)
@@ -24,6 +24,7 @@
 	  </link>
 	  <joint name="camera_joint" type="fixed">
-	    <axis xyz="-1 0 0" />
-	    <origin xyz="0.1935 0 0.012" rpy="0 0 0"/>
+	    <axis xyz="0 0 0" />
+	    <!--<origin xyz="0.1935 0 0.012" rpy="0 0 0"/>-->
+	    <origin xyz="-0.1920 0 0.012" rpy="3.14 3.14 0"/>
 	    <parent link="base_link"/>
 	    <child link="camera_link"/>

Commit message: Правки плагинов, моделей и лаунч-файлов  - в плагине использую AsyncSpinner вместо настройки очередей и потоков  - исправил колеса машинки, теперь она нормально ездит  - в twist_to_motors убрал MAX_PWM, пусть всегда будет 255  - чутка причесал launch-файлы

File: car_description/urdf/camera.xacro (robot description, xacro)
@@ -26,5 +26,4 @@
 	  </joint>
 	  <gazebo reference="camera_link">
-        <material>Gazebo/Red</material>
         <sensor type="camera" name="camera1">
 	      <update_rate>30.0</update_rate>

File: car_description/urdf/car.xacro (robot description, xacro)
@@ -8,10 +8,10 @@
     <xacro:property name="camera_size" value="0.03" />
     <xacro:body/>
-    <xacro:wheel parent="base_link" side="left" x_pos="${-wheel_stride}" name="wheel_1_left"/>
-    <xacro:wheel parent="base_link" side="right" x_pos="${-wheel_stride}" name="wheel_1_right"/>
-    <xacro:wheel parent="base_link" side="left" x_pos="0" name="wheel_2_left"/>
-    <xacro:wheel parent="base_link" side="right" x_pos="0" name="wheel_2_right"/>
-    <xacro:wheel parent="base_link" side="left" x_pos="${wheel_stride}" name="wheel_3_left"/>
-    <xacro:wheel parent="base_link" side="right" x_pos="${wheel_stride}" name="wheel_3_right"/>
+    <xacro:wheel parent="base_link" side="left"  x_pos="${-wheel_stride}" name="wheel_1_left"  z_offset="0.001"/>
+    <xacro:wheel parent="base_link" side="right" x_pos="${-wheel_stride}" name="wheel_1_right" z_offset="0.001"/>
+    <xacro:wheel parent="base_link" side="left"  x_pos="0"                name="wheel_2_left"  z_offset="0"/>
+    <xacro:wheel parent="base_link" side="right" x_pos="0"                name="wheel_2_right" z_offset="0"/>
+    <xacro:wheel parent="base_link" side="left"  x_pos="${wheel_stride}"  name="wheel_3_left"  z_offset="0.001"/>
+    <xacro:wheel parent="base_link" side="right" x_pos="${wheel_stride}"  name="wheel_3_right" z_offset="0.001"/>
     <xacro:my_camera/>
     <gazebo>

File: car_description/urdf/wheel.xacro (robot description, xacro)
@@ -1,5 +1,5 @@
 <?xml version="1.0"?>
 <robot xmlns:xacro="http://www.ros.org/wiki/xacro">
-    <xacro:macro name="wheel" params="parent side x_pos name">
+    <xacro:macro name="wheel" params="parent side x_pos name z_offset">
         <xacro:left_right side="${side}"/>
         <xacro:property name="wheel_width" value="0.06" />
@@ -26,7 +26,11 @@
             <parent link="${parent}"/>
             <child  link="${name}"/>
-            <origin xyz="${x_pos} ${x_sign*0.083} 0" rpy="0 0 0"/>
-            <axis xyz="0 -1 0"/>
+            <origin xyz="${x_pos} ${x_sign*0.083} ${z_offset}" rpy="0 0 0"/>
+            <axis xyz="0 1 0"/>
         </joint>
+        <!--<gazebo reference="${name}">
+            <mu1>50</mu1>
+            <mu2>50</mu2>
+        </gazebo>-->
     </xacro:macro>
 </robot>
